File: PCB/Klotz.kicad_sch (KiCad schematic)
At the start: 55 parts, among them SW1 MX_SW_HS, SW10 MX_SW_HS, SW11 MX_SW_HS, SW12 MX_SW_HS, SW13 MX_SW_HS, SW14 MX_SW_HS, SW15 MX_SW_HS, SW16 MX_SW_HS, SW17 MX_SW_HS, SW18 RotaryEncoder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

Commit message: Renames
Parts:
- BT1: footprint KLOTZ:JST_PH_reversible -> PLITKA:JST_PH_reversible
- BT2: footprint KLOTZ:custombatteryconnector -> PLITKA:custombatteryconnector
- D1, D10, D11, D12, D13, D14, D15, D16, D17, D2, D3, D4, D5, D6, D7, D8, D9: footprint KLOTZ:Diode_SOD123 -> PLITKA:Diode_SOD123
- JP1, JP3, JP4: footprint KLOTZ:Jumper -> PLITKA:Jumper; symbol KLOTZ:Device_Jumper_NO_Small -> PLITKA:Device_Jumper_NO_Small
- JP2: footprint KLOTZ:Jumper -> PLITKA:Jumper
- L1, L2, L3: footprint KLOTZ:LED_3mm_reversible -> PLITKA:LED_3mm_reversible
- PSW1: footprint KLOTZ:MSK12C02_reversible -> PLITKA:MSK12C02_reversible
- R1, R2, R3: footprint KLOTZ:R_1206_DoubleSided -> PLITKA:R_1206_DoubleSided
- SW1, SW2: footprint KLOTZ:Kailh_socket_PG1350_optional_reversible -> PLITKA:Kailh_socket_PG1350_optional_reversible; symbol KLOTZ:MX_SW_HS -> PLITKA:MX_SW_HS
- SW10, SW11, SW12, SW13, SW14, SW15, SW16, SW17, SW3, SW4, SW5, SW6, SW7, SW8, SW9: footprint KLOTZ:Kailh_socket_PG1350_optional_reversible -> PLITKA:Kailh_socket_PG1350_optional_reversible
- U1: footprint KLOTZ:ProMicro_v2 -> PLITKA:ProMicro_v2
Other:
- title: KLOTZ split keyboard -> PLITKA split keyboard
