File: PCB/PLITKA.kicad_sch (KiCad schematic)
At the start: 55 parts, among them SW1 MX_SW_HS, SW10 MX_SW_HS, SW11 MX_SW_HS, SW12 MX_SW_HS, SW13 MX_SW_HS, SW14 MX_SW_HS, SW15 MX_SW_HS, SW16 MX_SW_HS, SW17 MX_SW_HS, SW18 RotaryEncoder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

Commit message: KiCad versions update
Parts:
- RSW1: footprint (none) -> PLITKA:ResetSW
