File: PCB/PLITKA.kicad_pcb (KiCad board)
At the start: 2 copper layers, 120.5 x 85.5 mm, 56 parts, among them SW1 MX_SW_HS, SW10 MX_SW_HS, SW11 MX_SW_HS, SW12 MX_SW_HS, SW13 MX_SW_HS, SW14 MX_SW_HS, SW15 MX_SW_HS, SW16 MX_SW_HS, SW17 MX_SW_HS, SW18 RotaryEncoder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

Commit message: Encoder removal from pcb
Parts:
- removed SW18: RotaryEncoder, Rotary_Encoder:RotaryEncoder_Alps_EC12E_Vertical_H20mm
Connections:
- U1 pad 18: ENCB -> unconnected-(U1-F6/A1-Pad18)_1
- U1 pad 19: ENCA -> unconnected-(U1-F5/A2-Pad19)
Routing:
- net (no net): track 0.00 -> 70.7 mm, vias 0 -> 2
- net ENCA: track 42.4 -> 0.00 mm, vias 2 -> 0
- net ENCB: track 35.1 -> 0.00 mm, vias 2 -> 0
- net unconnected-(U1-2/D1/SDA-Pad5): track 17.1 -> 0.00 mm
- net unconnected-(U1-TX0/D3-Pad1)_1: track 17.1 -> 0.00 mm
- net unconnected-(U1-RX1/D2-Pad2): track 17.1 -> 0.00 mm
- net unconnected-(U1-F4/A3-Pad20)_1: track 14.3 -> 0.00 mm, vias 1 -> 0
- net unconnected-(PSW1A-A-Pad1): track 5.12 -> 0.00 mm, vias 1 -> 0
Other:
- board text removed: "--ENCA"
- board text removed: "--ENCB"
- board text removed: "ENCODER"
