File: PCB/pinky.kicad_sch (KiCad schematic)
At the start: 47 parts, among them SW1 SW_SPDT_321, SW10 MX_SW_HS, SW11 MX_SW_HS, SW12 MX_SW_HS, SW13 MX_SW_HS, SW14 MX_SW_HS, SW15 MX_SW_HS, SW16 MX_SW_HS, SW17 MX_SW_HS, SW18 MX_SW_HS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

Commit message: Keyboard renamed to Pinky, to reflect the idea in the name
Parts:
- JP1, JP3, JP4: symbol PLITKA:Device_Jumper_NO_Small -> Pinky:Device_Jumper_NO_Small
- SW1: footprint PLITKA:MSK12C02_reversible -> Pinky:MSK12C02_reversible
- SW10, SW11, SW12, SW13, SW14, SW15, SW16, SW17, SW18, SW2, SW3, SW4, SW5, SW6, SW7, SW8, SW9: footprint PLITKA:Kailh_socket_PG1350_optional_reversible -> Pinky:Kailh_socket_PG1350_optional_reversible; symbol PLITKA:MX_SW_HS -> Pinky:MX_SW_HS
- U1: footprint PLITKA:nice_nano -> Pinky:nice_nano; symbol PLITKA:nice_nano -> Pinky:nice_nano
Other:
- title: PLITKA keyboard -> Pinky keyboard

Commit message: Metadata clean up
Other:
- title: Pinky keyboard -> Pinky split keyboard
Changed lines of the file:
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@@
 	(paper "A5")
 	(title_block
-		(title "Pinky keyboard")
-		(date "12/06/2026")
+		(title "Pinky split keyboard")
+		(date "19/06/2026")
 		(rev "0.1")
 		(comment 1 "Author: rawrex")
