File: PCB/pinky.kicad_sch (KiCad schematic)
At the start: 47 parts, among them SW1 SW_SPDT_321, SW10 MX_SW_HS, SW11 MX_SW_HS, SW12 MX_SW_HS, SW13 MX_SW_HS, SW14 MX_SW_HS, SW15 MX_SW_HS, SW16 MX_SW_HS, SW17 MX_SW_HS, SW18 MX_SW_HS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

Commit message: Further symbols sync and clean up
Parts:
- SW1: footprint Pinky:MSK12C02_reversible -> (none)

Commit message: Symbol to footprint mapping
Parts:
- JP1: footprint (none) -> Pinky:Jumper
Changed lines of the file:
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@@
 			)
 		)
-		(property "Footprint" ""
+		(property "Footprint" "Pinky:Jumper"
 			(at 45.72 114.3 0)
 			(hide yes)

Commit message: Updates pull
Parts:
- JP2, JP3, JP4: footprint (none) -> Pinky:Jumper
Changed lines of the file:
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@@
 		)
 		(property "Value" "PWR_FLAG"
-			(at 53.34 83.82 90)
+			(at 48.26 83.82 0)
 			(show_name no)
 			(do_not_autoplace no)
@@
 			)
 		)
-		(property "Footprint" ""
+		(property "Footprint" "Pinky:Jumper"
 			(at 45.72 123.19 0)
 			(hide yes)
@@
 		)
 		(property "Value" "+BATT"
-			(at 37.338 35.56 90)
+			(at 40.894 35.56 0)
 			(show_name no)
 			(do_not_autoplace no)
@@
 		)
 		(property "Value" "GND"
-			(at 38.608 83.82 90)
+			(at 40.64 83.82 0)
 			(show_name no)
 			(do_not_autoplace no)
@@
 			)
 		)
-		(property "Footprint" ""
+		(property "Footprint" "Pinky:Jumper"
 			(at 45.72 127 0)
 			(hide yes)
@@
 			)
 		)
-		(property "Footprint" ""
+		(property "Footprint" "Pinky:Jumper"
 			(at 45.72 118.11 0)
 			(hide yes)
