File: PCB/pinky.kicad_sch (KiCad schematic)
At the start: 47 parts, among them SW10 Switch, SW11 Switch, SW12 Switch, SW13 Switch, SW14 Switch, SW15 Switch, SW16 Switch, SW17 Switch, SW18 Switch, SW2 Switch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

Commit message: Updates pull
Parts:
- renumbered RESET to RESET19, SW_PWR to SW_PWR1
Connections:
- net +BATT: now also SW_PWR1.3 (A)
- net GND: now also RESET19.1
- net PAD1: now also BT1.1 (+)
- net PAD2: now also BT1.2 (-)
- net RESET: now also RESET19.2
- net at JP2.2, JP3.2: now also SW_PWR1.2 (B)
Changed lines of the file:
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@@
 	)
 	(junction
+		(at 50.8 120.65)
+		(diameter 0)
+		(color 0 0 0 0)
+	)
+	(junction
 		(at 110.49 77.47)
 		(diameter 0)
@@
 	)
 	(junction
-		(at 50.8 120.65)
-		(diameter 0)
-		(color 0 0 0 0)
-	)
-	(junction
 		(at 93.98 48.26)
 		(diameter 0)
@@
 	)
 	(no_connect
-		(at 64.77 123.19)
+		(at 62.23 123.19)
 	)
 	(no_connect
@@
 	(wire
 		(pts
-			(xy 48.26 114.3) (xy 55.88 114.3)
+			(xy 48.26 114.3) (xy 50.8 114.3)
 		)
 		(stroke
@@
 	(wire
 		(pts
-			(xy 48.26 127) (xy 55.88 127)
+			(xy 48.26 127) (xy 50.8 127)
 		)
 		(stroke
@@
 	(wire
 		(pts
-			(xy 67.31 118.11) (xy 64.77 118.11)
-		)
-		(stroke
-			(width 0)
-			(type default)
-		)
-	)
-	(wire
-		(pts
 			(xy 105.41 67.31) (xy 105.41 85.09)
 		)
@@
 	(wire
 		(pts
-			(xy 50.8 120.65) (xy 54.61 120.65)
+			(xy 50.8 120.65) (xy 52.07 120.65)
 		)
 		(stroke
@@
 	(wire
 		(pts
-			(xy 55.88 114.3) (xy 55.88 113.03)
+			(xy 50.8 114.3) (xy 50.8 113.03)
 		)
 		(stroke
@@
 	(wire
 		(pts
-			(xy 55.88 127) (xy 55.88 128.27)
+			(xy 50.8 127) (xy 50.8 128.27)
 		)
 		(stroke
@@
 	(symbol
 		(lib_id "power:+BATT")
-		(at 67.31 118.11 270)
+		(at 62.23 118.11 270)
 		(unit 1)
 		(body_style 1)
@@
 		(dnp no)
 		(property "Reference" "#PWR6"
-			(at 63.5 118.11 0)
+			(at 58.42 118.11 0)
 			(hide yes)
 			(show_name no)
@@
 		)
 		(property "Value" "+BATT"
-			(at 70.866 118.11 0)
+			(at 65.786 118.11 0)
 			(show_name no)
 			(do_not_autoplace no)
@@
 		)
 		(property "Footprint" ""
-			(at 67.31 118.11 0)
+			(at 62.23 118.11 0)
 			(hide yes)
 			(show_name no)
@@
 		)
 		(property "Datasheet" ""
-			(at 67.31 118.11 0)
+			(at 62.23 118.11 0)
 			(hide yes)
 			(show_name no)
@@
 		)
 		(property "Description" "Power symbol creates a global label with name \"+BATT\""
-			(at 67.31 118.11 0)
+			(at 62.23 118.11 0)
 			(hide yes)
 			(show_name no)
@@
 	(symbol
 		(lib_id "Pinky:MSK12C02")
-		(at 59.69 120.65 0)
+		(at 57.15 120.65 0)
 		(unit 1)
 		(body_style 1)
@@
 		(in_pos_files yes)
 		(dnp no)
-		(property "Reference" "SW_PWR"
-			(at 59.69 115.57 0)
+		(property "Reference" "SW_PWR1"
+			(at 57.658 115.316 0)
 			(show_name no)
 			(do_not_autoplace no)
@@
 		)
 		(property "Value" "MSK12C02"
-			(at 59.69 125.73 0)
+			(at 57.15 125.73 0)
 			(hide yes)
 			(show_name no)
@@
 		)
 		(property "Footprint" "Pinky:MSK12C02"
-			(at 59.69 130.81 0)
+			(at 57.15 130.81 0)
 			(hide yes)
 			(show_name no)
@@
 		)
 		(property "Datasheet" ""
-			(at 59.69 128.27 0)
+			(at 57.15 128.27 0)
 			(hide yes)
 			(show_name no)
@@
 		)
 		(property "Description" "Switch, single pole double throw"
-			(at 59.69 120.65 0)
+			(at 57.15 120.65 0)
 			(hide yes)
 			(show_name no)
@@
 			(project "pinky"
 				(path "/231ead31-262f-44fe-a25c-f58d2465dcca"
-					(reference "SW1")
+					(reference "SW_PWR1")
 					(unit 1)
 				)
@@
 			)
 		)
-		(property "Sim.Device" "V"
-			(at 33.02 121.92 0)
-			(hide yes)
-			(show_name no)
-			(do_not_autoplace no)
-			(effects
-				(font
-					(size 1.27 1.27)
-				)
-			)
-		)
-		(property "Sim.Type" "DC"
-			(at 33.02 121.92 0)
-			(hide yes)
-			(show_name no)
-			(do_not_autoplace no)
-			(effects
-				(font
-					(size 1.27 1.27)
-				)
-			)
-		)
-		(property "Sim.Pins" "1=+ 2=-"
-			(at 33.02 121.92 0)
-			(hide yes)
-			(show_name no)
-			(do_not_autoplace no)
-			(effects
-				(font
-					(size 1.27 1.27)
-				)
-			)
-		)
 		(pin "1"
 		)
@@
 		(dnp no)
 		(fields_autoplaced yes)
-		(property "Reference" "RESET"
+		(property "Reference" "RESET19"
 			(at 175.26 77.47 0)
+			(hide yes)
 			(show_name no)
 			(do_not_autoplace no)
@@
 			(project "pinky"
 				(path "/231ead31-262f-44fe-a25c-f58d2465dcca"
-					(reference "SW19")
+					(reference "RESET19")
 					(unit 1)
 				)
@@
 	(symbol
 		(lib_id "power:GND")
-		(at 55.88 128.27 0)
+		(at 50.8 128.27 0)
 		(unit 1)
 		(body_style 1)
@@
 		(fields_autoplaced yes)
 		(property "Reference" "#PWR1"
-			(at 55.88 134.62 0)
+			(at 50.8 134.62 0)
 			(hide yes)
 			(show_name no)
@@
 		)
 		(property "Value" "GND"
-			(at 55.88 133.35 0)
+			(at 50.8 133.35 0)
 			(show_name no)
 			(do_not_autoplace no)
@@
 		)
 		(property "Footprint" ""
-			(at 55.88 128.27 0)
+			(at 50.8 128.27 0)
 			(hide yes)
 			(show_name no)
@@
 		)
 		(property "Datasheet" ""
-			(at 55.88 128.27 0)
+			(at 50.8 128.27 0)
 			(hide yes)
 			(show_name no)
@@
 		)
 		(property "Description" "Power symbol creates a global label with name \"GND\" , ground"
-			(at 55.88 128.27 0)
+			(at 50.8 128.27 0)
 			(hide yes)
 			(show_name no)
@@
 	(symbol
 		(lib_id "power:GND")
-		(at 55.88 113.03 180)
+		(at 50.8 113.03 180)
 		(unit 1)
 		(body_style 1)
@@
 		(fields_autoplaced yes)
 		(property "Reference" "#PWR2"
-			(at 55.88 106.68 0)
+			(at 50.8 106.68 0)
 			(hide yes)
 			(show_name no)
@@
 		)
 		(property "Value" "GND"
-			(at 55.88 107.95 0)
+			(at 50.8 107.95 0)
 			(show_name no)
 			(do_not_autoplace no)
@@
 		)
 		(property "Footprint" ""
-			(at 55.88 113.03 0)
+			(at 50.8 113.03 0)
 			(hide yes)
 			(show_name no)
@@
 		)
 		(property "Datasheet" ""
-			(at 55.88 113.03 0)
+			(at 50.8 113.03 0)
 			(hide yes)
 			(show_name no)
@@
 		)
 		(property "Description" "Power symbol creates a global label with name \"GND\" , ground"
-			(at 55.88 113.03 0)
+			(at 50.8 113.03 0)
 			(hide yes)
 			(show_name no)
