File: PCB/pinky.kicad_pcb (KiCad board)
At the start: 2 copper layers, 54 parts, among them SW10 Switch, SW11 Switch, SW12 Switch, SW13 Switch, SW14 Switch, SW15 Switch, SW16 Switch, SW17 Switch, SW18 Switch, SW2 Switch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

Commit message: Routes clean up
Routing:
- net col_A: track 122.0 -> 92.3 mm
- net row_D: track 65.3 -> 40.6 mm
- net col_D: track 139.4 -> 118.3 mm
- net row_A: track 152.3 -> 145.5 mm
- net col_B: track 135.4 -> 128.8 mm
- net row_B: track 112.7 -> 107.7 mm
- net Net-(D14-A): track 32.6 -> 28.9 mm
- net row_C: track 92.2 -> 91.0 mm
- net col_C: track 97.4 -> 98.4 mm
